Commit message: Prepare OneRobotics A1 contribution

File: source/h1_reach/h1_reach/assets/urdf/A1/a1_left.urdf (robot description, URDF)
Before this commit: robot a1_l_urdf, 9 links, 8 joints
Links:
- link Link1: geometry collision mesh filename=../../meshes/A1/A1_l/Link_L1.STL; visual mesh filename=../../meshes/A1/A1_l/Link_L1.STL
- link Link2: geometry collision mesh filename=../../meshes/A1/A1_l/Link_L2.STL; visual mesh filename=../../meshes/A1/A1_l/Link_L2.STL
- link Link3: geometry collision mesh filename=../../meshes/A1/A1_l/Link_L3.STL; visual mesh filename=../../meshes/A1/A1_l/Link_L3.STL
- link Link4: geometry collision mesh filename=../../meshes/A1/A1_l/Link_L4.STL; visual mesh filename=../../meshes/A1/A1_l/Link_L4.STL
- link Link5: geometry collision mesh filename=../../meshes/A1/A1_l/Link_L5.STL; visual mesh filename=../../meshes/A1/A1_l/Link_L5.STL
- link Link6: geometry collision mesh filename=../../meshes/A1/A1_l/Link_L6.STL; visual mesh filename=../../meshes/A1/A1_l/Link_L6.STL
- link Link7: geometry collision mesh filename=../../meshes/A1/A1_l/Link_L7.STL; visual mesh filename=../../meshes/A1/A1_l/Link_L7.STL
- link base_link: geometry collision mesh filename=../../meshes/A1/A1_l/base_link.STL; visual mesh filename=../../meshes/A1/A1_l/base_link.STL

File: source/h1_reach/h1_reach/assets/urdf/A1/a1_right.urdf (robot description, URDF)
Before this commit: robot a1_r_urdf, 8 links, 7 joints
Links:
- link Link1: geometry collision mesh filename=../../meshes/A1/A1_r/Link_R1.STL; visual mesh filename=../../meshes/A1/A1_r/Link_R1.STL
- link Link2: geometry collision mesh filename=../../meshes/A1/A1_r/Link_R2.STL; visual mesh filename=../../meshes/A1/A1_r/Link_R2.STL
- link Link3: geometry collision mesh filename=../../meshes/A1/A1_r/Link_R3.STL; visual mesh filename=../../meshes/A1/A1_r/Link_R3.STL
- link Link4: geometry collision mesh filename=../../meshes/A1/A1_r/Link_R4.STL; visual mesh filename=../../meshes/A1/A1_r/Link_R4.STL
- link Link5: geometry collision mesh filename=../../meshes/A1/A1_r/Link_R5.STL; visual mesh filename=../../meshes/A1/A1_r/Link_R5.STL
- link Link6: geometry collision mesh filename=../../meshes/A1/A1_r/Link_R6.STL; visual mesh filename=../../meshes/A1/A1_r/Link_R6.STL
- link Link7: geometry collision mesh filename=../../meshes/A1/A1_r/Link_R7.STL; visual mesh filename=../../meshes/A1/A1_r/Link_R7.STL
- link base_link: geometry collision mesh filename=../../meshes/A1/A1_r/base_link.STL; visual mesh filename=../../meshes/A1/A1_r/base_link.STL

File: source/h1_reach/h1_reach/assets/urdf/A1_dual/A1_dual.urdf (robot description, URDF)
Before this commit: robot A1_dual, 18 links, 17 joints
Links:
- link base_link: geometry collision mesh filename=../../meshes/A1_dual/base_link.STL; visual mesh filename=../../meshes/A1_dual/base_link.STL
- link left_base_link: geometry collision mesh filename=../../meshes/A1_dual/Link_base_L.STL; visual mesh filename=../../meshes/A1_dual/Link_base_L.STL
- link left_link1: geometry collision mesh filename=../../meshes/A1_dual/Link_L1.STL; visual mesh filename=../../meshes/A1_dual/Link_L1.STL
- link left_link2: geometry collision mesh filename=../../meshes/A1_dual/Link_L2.STL; visual mesh filename=../../meshes/A1_dual/Link_L2.STL
- link left_link3: geometry collision mesh filename=../../meshes/A1_dual/Link_L3.STL; visual mesh filename=../../meshes/A1_dual/Link_L3.STL
- link left_link4: geometry collision mesh filename=../../meshes/A1_dual/Link_L4.STL; visual mesh filename=../../meshes/A1_dual/Link_L4.STL
- link left_link5: geometry collision mesh filename=../../meshes/A1_dual/Link_L5.STL; visual mesh filename=../../meshes/A1_dual/Link_L5.STL
- link left_link6: geometry collision mesh filename=../../meshes/A1_dual/Link_L6.STL; visual mesh filename=../../meshes/A1_dual/Link_L6.STL
- link left_link7: geometry collision mesh filename=../../meshes/A1_dual/Link_L7.STL; visual mesh filename=../../meshes/A1_dual/Link_L7.STL
- link right_base_link: geometry collision mesh filename=../../meshes/A1_dual/Link_base_R.STL; visual mesh filename=../../meshes/A1_dual/Link_base_R.STL
- link right_link1: geometry collision mesh filename=../../meshes/A1_dual/Link_R1.STL; visual mesh filename=../../meshes/A1_dual/Link_R1.STL
- link right_link2: geometry collision mesh filename=../../meshes/A1_dual/Link_R2.STL; visual mesh filename=../../meshes/A1_dual/Link_R2.STL
- link right_link3: geometry collision mesh filename=../../meshes/A1_dual/Link_R3.STL; visual mesh filename=../../meshes/A1_dual/Link_R3.STL
- link right_link4: geometry collision mesh filename=../../meshes/A1_dual/Link_R4.STL; visual mesh filename=../../meshes/A1_dual/Link_R4.STL
- link right_link5: geometry collision mesh filename=../../meshes/A1_dual/Link_R5.STL; visual mesh filename=../../meshes/A1_dual/Link_R5.STL
- link right_link6: geometry collision mesh filename=../../meshes/A1_dual/Link_R6.STL; visual mesh filename=../../meshes/A1_dual/Link_R6.STL
- link right_link7: geometry collision mesh filename=../../meshes/A1_dual/Link_R7.STL; visual mesh filename=../../meshes/A1_dual/Link_R7.STL
